File: nrf.kicad_sch (KiCad schematic)
At the start: 32 parts, among them J1 USB_C_Receptacle_USB2.0_16P, Q1 lpo404, SW1 RESET, U1 nRF52840, U2 BQ25101YFPR, Y1 32.768kHz, Y2 32mHz

Commit message: Dodanie komponentów do kontrolera baterii oraz przypisanie kilku lini.
Parts:
- added C17: 2.2uF, symbol Device:C_Small
- added R10, R11: 33R, Resistor_THT:R_Array_SIP4, symbol Device:R_Small
- added R6, R7: 2.7k, symbol Device:R_Small
- added R8: 1M, symbol Device:R_Small
- added R9: 510k, symbol Device:R_Small
- added TP1: BAT0, Package_SO:TSSOP-20_4.4x6.5mm_P0.65mm, symbol Connector:TestPoint
- added TP2: GND0, Package_SO:TSSOP-20_4.4x6.5mm_P0.65mm, symbol Connector:TestPoint
Connections:
- net +BATT: now also U2.A1 (OUT), C17.2, R8.1, TP1.1
- net GND: now also U2.C1 (CHG_N), C17.1, R6.2, TP2.1
- net USBD+: now also R11.2; no longer U1.AD6 (D+)
- net USBD-: now also R10.2; no longer U1.AD4 (D-)
- net P0.31_AIN7_BAT: now reaches U1.A8 (AIN7/P0.31)
- net P0.31_AIN7_BAT: now also R8.2, R9.1
- net P0.14_READ_BAT: now reaches U1.AC9 (P0.14)
- net P0.14_READ_BAT: now also R9.2
- net P0.13_HICHG: now reaches U1.AD8 (P0.13)
- net P0.13_HICHG: now also R7.2
- net at U2.B2 (ISET): now also R6.1, R7.1
- new net: R11.1, U1.AD6 (D+)
- new net: R10.1, U1.AD4 (D-)
Other:
- moved on the sheet: C14, C5, C7, C9, R5, U2

Commit message: Dodanie ledu
Parts:
- added D1: LED_BGRA, symbol Device:LED_BGRA
- added D2: CHG0, symbol Device:LED
- added R12, R13, R15: 2.2k, symbol Device:R_Small
- added R14: 10k, symbol Device:R_Small
Connections:
- net +3.3V: now also D1.4 (A), R15.1
- net GND: now also D2.1 (K)
- new net: D2.2 (A), R15.2
- new net: D1.1 (BK), R13.1
- new net: D1.2 (GK), R14.2
- new net: D1.3 (RK), R12.1
- new net P0.06_LED_BLUE: R13.2
- new net P0.26_LED_RED: R12.2
- new net P0.30_LED_GREEN: R14.1
Other:
- note added: "LED"
- moved on the sheet: C15, C16, C17, C7, CR1, Q1, R4, R5, R6, R7, R8, R9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
